File: KiCAD/WeighingScalePCB/_autosave-WeighingScalePCB.kicad_sch (KiCad schematic)
At the start: 56 parts, among them IC1 MAX6675ISA+T, IC2 APS11753KMDALX-9PL5, J1 Conn_01x04_Pin, J2 AudioJack4, J3 CONN_14_FFC/FPC, J4 Battery Conn, Q1 MMBT2222A, Q2 NX138AKR, Q3 NX138AKR, Q4 NX138AKR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

Commit message: added components to library
Parts:
- removed U4: 74HC74, symbol 74xx:74HC74
- removed U7: 74AHC1G08, symbol 74xGxx:74AHC1G08
- removed U8: 74AHC1G04, symbol 74xGxx:74AHC1G04
- removed U9: NE555D, Package_SO:SOIC-8_3.9x4.9mm_P1.27mm, symbol Timer:NE555D
- J1: footprint Connector_PinHeader_1.00mm:PinHeader_1x04_P1.00mm_Vertical -> Connector_JST:JST_SH_SM04B-SRSS-TB_1x04-1MP_P1.00mm_Horizontal
- J4: footprint (none) -> Connector_TE-Connectivity:TE_440055-2_1x02_P2.00mm_Horizontal
Connections:
- net Time is gone; now on net Tare: U1.4 (GPIO21_D3)
- net beep trigger is gone; now on an unnamed net: Q4.1 (G)
- net Tare: now also D2.2 (A), U5.1 (Q), U6.1 (Q)
Other:
- moved on the sheet: C1, C15, C16, C17, C2, C3, C4, C5, C6, C7, C8, C9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
